File: extension/Main.kicad_sch (KiCad schematic)
At the start: 37 parts, among them IC501 DA7212-01UM2, IC502 MAX32664, IC503 MAX86141, IC504 LIS2DS12, X501 MB1, X502 MB2, Y501 32kHz

Commit message: First version done
Parts:
- added C522: 100n, Capacitor_SMD:C_0201_0603Metric, symbol Device:C_Small
- C509, C512, C513, C517: footprint Capacitor_SMD:C_0402_1005Metric -> Capacitor_SMD:C_0201_0603Metric; manf# 04023D105KAT2A -> 02016W105MAT2A; mouser# 581-04023D105KAT2A -> 581-02016W105MAT2A
- C514, C515, C516, C518, C519, C520, C521: footprint Capacitor_SMD:C_0402_1005Metric -> Capacitor_SMD:C_0201_0603Metric
- FB501, FB502: footprint Inductor:L0402 -> Inductor_SMD:L_0402_1005Metric
- IC501: manf (none) -> Renesas / Dialog; manf# (none) -> DA7212-01UM2; mouser# (none) -> 724-DA7212-01UM2
- R501: footprint Resistor_SMD:R_0402_1005Metric -> Resistor_SMD:R_0201_0603Metric; manf# CR0402-JW-103GLF -> CR0201-JW-103GLF; mouser# 652-CR0402-JW-103GLF -> 652-CR0201-JW-103GLF
- R502: footprint Resistor_SMD:R_0402_1005Metric -> Inductor_SMD:L_0201_0603Metric; manf YAGEO -> Vishay; manf# RC0402FR-7D4K7L -> CRCW020147K5FNED; mouser# 603-RC0402FR-7D4K7L -> 71-CRCW020147K5FNED
- R503: value R_Small -> 0R; manf (none) -> YAGEO; manf# (none) -> 603-RC0201FR-SNE96L; mouser# (none) -> RC0201FR-SNE96L
- R504: footprint Resistor_SMD:R_0402_1005Metric -> Resistor_SMD:R_0201_0603Metric
Connections:
- net +1V8: now also X501.11 (Pin_11); no longer X502.1 (Pin_1)
- net GND: now also X501.14 (Pin_14), X501.2 (Pin_2), X501.4 (Pin_4), X502.13 (Pin_13), C522.1; no longer X501.7 (Pin_7), X502.14 (Pin_14)
- net GNDA: now also C522.2
- net I2S_BCLK: now also X501.5 (Pin_5); no longer X501.2 (Pin_2)
- net I2S_DIN: now also X501.7 (Pin_7); no longer X501.1 (Pin_1)
- net I2S_MCLK: now also X501.1 (Pin_1); no longer X501.4 (Pin_4)
- net SCL: now also X502.12 (Pin_12); no longer X502.9 (Pin_9)
- net SDA: now also X502.10 (Pin_10); no longer X502.8 (Pin_8)
- net SP-N: now also X501.10 (Pin_10), X501.12 (Pin_12); no longer X501.13 (Pin_13), X501.14 (Pin_14)
- net SP-P: now also X501.6 (Pin_6), X501.8 (Pin_8); no longer X501.11 (Pin_11), X501.12 (Pin_12)
- net STATUS: now also X502.14 (Pin_14); no longer X502.11 (Pin_11)
- net VSYS: now also X502.1 (Pin_1); no longer X502.2 (Pin_2)
- net V_{DD}: now also X502.4 (Pin_4); no longer X502.3 (Pin_3)
- net ~{RESET_{HR}}: now also X502.11 (Pin_11); no longer X502.10 (Pin_10)
- no-connect marks 26 -> 24
