File: extension/ZSWatch-Extension.kicad_pcb (KiCad board)
At the start: 4 copper layers, 16.8 x 16.8 mm, 37 parts, among them IC501 MAX32664, IC502 LIS2DS12, IC503 MAX86141, IC601 DA7212-01UM2, X701 MB2, X702 MB1, Y501 32kHz

Commit message: Update outputs (release)
Other:
- board text added: "0.035mm (1.00oz)"
- board text added: "0.196mm"
- board text added: "0.43mm"
- board text added: "GND"
- board text added: "Plane"
- board text added: "Prepreg"
- board text added: "Supply"
- board text added: "Total thickness: 0.982mm"
- board text removed: "0.035mm (1oz)"
- board text removed: "1.51mm"
- board text removed: "Total thickness: 1.6mm"
