File: extension/Audio.kicad_sch (KiCad schematic)
At the start: 15 parts, among them IC601 DA7212-01UM2

Commit message: Prepare release 1.0.0
Signed-off-by: Daniel Kampert <danielkampert@kampis-elektroecke.de>
Other:
- title: Audio -> (none)
Changed lines of the file:
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@@
 	(paper "A4")
 	(title_block
-		(title "Audio")
 		(date "2025-07-13")
 		(rev "${REVISION}")
