File: extension/Block Diagram.kicad_sch (KiCad schematic)
At the start: 0 parts

Commit message: Prepare release 1.0.0
Signed-off-by: Daniel Kampert <danielkampert@kampis-elektroecke.de>
Other:
- title: Block-Diagram -> Block Diagram
Changed lines of the file:
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@@
 	(paper "A3")
 	(title_block
-		(title "Block-Diagram")
+		(title "Block Diagram")
 		(date "2025-07-13")
 		(rev "${REVISION}")
