File: extension/Power - Topology.kicad_sch (KiCad schematic)
At the start: 0 parts

Commit message: Prepare release 1.0.0
Signed-off-by: Daniel Kampert <danielkampert@kampis-elektroecke.de>
Other:
- title: (none) -> Power - Topology
Changed lines of the file:
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@@
 	(paper "A3")
 	(title_block
+		(title "Power - Topology")
 		(date "2025-07-13")
 		(rev "${REVISION}")
@@
 		)
 	)
+	(text_box "[${#}] ${TITLE}"
+		(exclude_from_sim no)
+		(at 12.7 12.7 0)
+		(size 393.7 27.94)
+		(margins 4.4999 4.4999 4.4999 4.4999)
+		(stroke
+			(width -0.0001)
+			(type default)
+		)
+		(fill
+			(type none)
+		)
+		(effects
+			(font
+				(face "Times New Roman")
+				(size 6 6)
+				(thickness 1.2)
+				(bold yes)
+				(color 162 22 34 1)
+			)
+		)
+	)
 	(text_box "Spec 2"
 		(exclude_from_sim no)
@@
 	)
 	(image
-		(at 214.63 120.65)
+		(at 212.09 146.05)
 		(scale 1.51331)
 		(data "iVBORw0KGgoAAAANSUhEUgAAC0QAAAWQCAYAAADApWVoAAAABHNCSVQICAgIfAhkiAAAIABJREFU"
