File: extension/ZSWatch-Extension.kicad_sch (KiCad schematic)
At the start: 0 parts

Commit message: Prepare release 1.0.0
Signed-off-by: Daniel Kampert <danielkampert@kampis-elektroecke.de>
Other:
- title: Extension-HW -> (none)
Changed lines of the file:
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@@
 	(paper "A3")
 	(title_block
-		(title "Extension-HW")
 		(date "2025-07-13")
 		(rev "${REVISION}")
